Commit message: reconstructing legged_estimator

File: src/legged_description/resource/anymal_c/urdf/anymal.urdf (robot description, URDF)
Before this commit: robot anymal, 78 links, 77 joints
Links:
- link LF_FOOT: geometry collision cylinder length=0.282504 radius=0.0175; collision sphere radius=0.03
- link LF_HAA: geometry visual mesh filename=package://legged_description/resource/anymal_c/meshes/drive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 scale=1.0 1.0 1.0
- link LF_HFE: geometry collision cylinder length=0.14 radius=0.05; visual mesh filename=package://legged_description/resource/anymal_c/meshes/drive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 scale=1.0 1.0 1.0
- link LF_KFE: geometry collision cylinder length=0.14 radius=0.05; visual mesh filename=package://legged_description/resource/anymal_c/meshes/drive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 scale=1.0 1.0 1.0
- link LF_hip_fixed: geometry visual mesh filename=package://legged_description/resource/anymal_c/meshes/hip_l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 scale=1.0 1.0 1.0
- link LF_shank_fixed: geometry collision box size=0.114998 0.0675 0.04; collision cylinder length=0.04 radius=0.06
- link LF_thigh_fixed: geometry collision box size=0.075 0.06 0.282627; collision cylinder length=0.08 radius=0.065
- link LH_FOOT: geometry collision cylinder length=0.282504 radius=0.0175; collision sphere radius=0.03
- link LH_HAA: geometry visual mesh filename=package://legged_description/resource/anymal_c/meshes/drive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 scale=1.0 1.0 1.0
- link LH_HFE: geometry collision cylinder length=0.14 radius=0.05; visual mesh filename=package://legged_description/resource/anymal_c/meshes/drive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 scale=1.0 1.0 1.0
- link LH_KFE: geometry collision cylinder length=0.14 radius=0.05; visual mesh filename=package://legged_description/resource/anymal_c/meshes/drive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 scale=1.0 1.0 1.0
- link LH_hip_fixed: geometry visual mesh filename=package://legged_description/resource/anymal_c/meshes/hip_r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 scale=1.0 1.0 1.0
- link LH_shank_fixed: geometry collision box size=0.114998 0.0675 0.04; collision cylinder length=0.04 radius=0.06
- link LH_thigh_fixed: geometry collision box size=0.075 0.06 0.282627; collision cylinder length=0.08 radius=0.065
- link RF_FOOT: geometry collision cylinder length=0.282504 radius=0.0175; collision sphere radius=0.03
- link RF_HAA: geometry visual mesh filename=package://legged_description/resource/anymal_c/meshes/drive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 scale=1.0 1.0 1.0
- link RF_HFE: geometry collision cylinder length=0.14 radius=0.05; visual mesh filename=package://legged_description/resource/anymal_c/meshes/drive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 scale=1.0 1.0 1.0
- link RF_KFE: geometry collision cylinder length=0.14 radius=0.05; visual mesh filename=package://legged_description/resource/anymal_c/meshes/drive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 scale=1.0 1.0 1.0
- link RF_hip_fixed: geometry visual mesh filename=package://legged_description/resource/anymal_c/meshes/hip_r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 scale=1.0 1.0 1.0
- link RF_shank_fixed: geometry collision box size=0.114998 0.0675 0.04; collision cylinder length=0.04 radius=0.06
- link RF_thigh_fixed: geometry collision box size=0.075 0.06 0.282627; collision cylinder length=0.08 radius=0.065
- link RH_FOOT: geometry collision cylinder length=0.282504 radius=0.0175; collision sphere radius=0.03
- link RH_HAA: geometry visual mesh filename=package://legged_description/resource/anymal_c/meshes/drive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 scale=1.0 1.0 1.0
- link RH_HFE: geometry collision cylinder length=0.14 radius=0.05; visual mesh filename=package://legged_description/resource/anymal_c/meshes/drive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 scale=1.0 1.0 1.0
- link RH_KFE: geometry collision cylinder length=0.14 radius=0.05; visual mesh filename=package://legged_description/resource/anymal_c/meshes/drive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 scale=1.0 1.0 1.0
- link RH_hip_fixed: geometry visual mesh filename=package://legged_description/resource/anymal_c/meshes/hip_l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 scale=1.0 1.0 1.0
- link RH_shank_fixed: geometry collision box size=0.114998 0.0675 0.04; collision cylinder length=0.04 radius=0.06
- link RH_thigh_fixed: geometry collision box size=0.075 0.06 0.282627; collision cylinder length=0.08 radius=0.065
- link base: geometry collision box size=0.58 0.14 0.18; collision cylinder length=0.145 radius=0.09
- link battery: geometry visual mesh filename=package://legged_description/resource/anymal_c/meshes/batte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 scale=1.0 1.0 1.0
- link bottom_shell: geometry visual mesh filename=package://legged_description/resource/anymal_c/meshes/botto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 scale=1.0 1.0 1.0
- link depth_camera_front_camera: geometry visual mesh filename=package://legged_description/resource/anymal_c/meshes/depth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 scale=1.0 1.0 1.0
- link depth_camera_left_camera: geometry visual mesh filename=package://legged_description/resource/anymal_c/meshes/depth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 scale=1.0 1.0 1.0
- link depth_camera_rear_camera: geometry visual mesh filename=package://legged_description/resource/anymal_c/meshes/depth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 scale=1.0 1.0 1.0
- link depth_camera_right_camera: geometry visual mesh filename=package://legged_description/resource/anymal_c/meshes/depth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 scale=1.0 1.0 1.0
- link face_front: geometry collision box size=0.11 0.14 0.18; collision cylinder length=0.11 radius=0.09
- link face_rear: geometry collision box size=0.11 0.14 0.18; collision cylinder length=0.11 radius=0.09
- link handle: geometry visual mesh filename=package://legged_description/resource/anymal_c/meshes/handl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 scale=1.0 1.0 1.0
- link hatch: geometry visual mesh filename=package://legged_description/resource/anymal_c/meshes/hatch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 scale=1.0 1.0 1.0
- link lidar: geometry visual mesh filename=package://legged_description/resource/anymal_c/meshes/lidar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
- link lidar_cage: geometry collision cylinder length=0.12 radius=0.07; visual mesh filename=package://legged_description/resource/anymal_c/meshes/lidar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 scale=1.0 1.0 1.0
- link remote: geometry visual mesh filename=package://legged_description/resource/anymal_c/meshes/remot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 scale=1.0 1.0 1.0
- link top_shell: geometry visual mesh filename=package://legged_description/resource/anymal_c/meshes/top_s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 scale=1.0 1.0 1.0
- link wide_angle_camera_front_camera: geometry visual mesh filename=package://legged_description/resource/anymal_c/meshes/wide_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 scale=1.0 1.0 1.0
- link wide_angle_camera_rear_camera: geometry visual mesh filename=package://legged_description/resource/anymal_c/meshes/wide_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 scale=1.0 1.0 1.0

File: src/legged_description/resource/anymal_c/urdf/joint_gz.xacro (robot description, xacro)
@@ -1,20 +1,11 @@
 <?xml version="1.0"?>
 <robot xmlns:xacro="http://www.ros.org/wiki/xacro">
-  <xacro:macro name="leggedbot_base">
+  <xacro:macro name="leggedbot_base" params="name">
     <!-- 关节宏，复用接口定义 -->
     <xacro:macro name="leg_joint" params="name">
       <joint name="${name}">
-        <command_interface name="position">
-          <param name="min">-1</param>
-          <param name="max">1</param>
-        </command_interface>
-        <command_interface name="velocity">
-          <param name="min">-1</param>
-          <param name="max">1</param>
-        </command_interface>
-        <command_interface name="effort">
-          <param name="min">-1</param>
-          <param name="max">1</param>
-        </command_interface>
+        <command_interface name="position"/>
+        <command_interface name="velocity"/>
+        <command_interface name="effort"/>
         <state_interface name="position"/>
         <state_interface name="velocity"/>
@@ -24,7 +15,6 @@
     <ros2_control name="${name}" type="system">
         <hardware>
-            <plugin>legged_robot/LeggedBotBaseMotors</plugin>
+            <plugin>gz_ros2_control/GazeboSimSystem</plugin>
         </hardware>
-        <!-- 根据需要启用/禁用对应关节 -->
         <xacro:leg_joint name="LF_HAA"/>
         <xacro:leg_joint name="LF_HFE"/>
