Commit message: add lauch files

File: src/legged_bringup/resource/anymal_c/urdf/anymal.urdf (robot description, URDF)
Before this commit: robot anymal, 78 links, 77 joints
Links:
- link LF_FOOT: geometry collision cylinder length=0.282504 radius=0.0175; collision sphere radius=0.03
- link LF_HAA: geometry visual mesh filename=package://legged_bringup/resource/anymal_c/meshes/drive.dae scale=1.0 1.0 1.0
- link LF_HFE: geometry collision cylinder length=0.14 radius=0.05; visual mesh filename=package://legged_bringup/resource/anymal_c/meshes/drive.dae scale=1.0 1.0 1.0
- link LF_KFE: geometry collision cylinder length=0.14 radius=0.05; visual mesh filename=package://legged_bringup/resource/anymal_c/meshes/drive.dae scale=1.0 1.0 1.0
- link LF_hip_fixed: geometry visual mesh filename=package://legged_bringup/resource/anymal_c/meshes/hip_l.dae scale=1.0 1.0 1.0
- link LF_shank_fixed: geometry collision box size=0.114998 0.0675 0.04; collision cylinder length=0.04 radius=0.06
- link LF_thigh_fixed: geometry collision box size=0.075 0.06 0.282627; collision cylinder length=0.08 radius=0.065
- link LH_FOOT: geometry collision cylinder length=0.282504 radius=0.0175; collision sphere radius=0.03
- link LH_HAA: geometry visual mesh filename=package://legged_bringup/resource/anymal_c/meshes/drive.dae scale=1.0 1.0 1.0
- link LH_HFE: geometry collision cylinder length=0.14 radius=0.05; visual mesh filename=package://legged_bringup/resource/anymal_c/meshes/drive.dae scale=1.0 1.0 1.0
- link LH_KFE: geometry collision cylinder length=0.14 radius=0.05; visual mesh filename=package://legged_bringup/resource/anymal_c/meshes/drive.dae scale=1.0 1.0 1.0
- link LH_hip_fixed: geometry visual mesh filename=package://legged_bringup/resource/anymal_c/meshes/hip_r.dae scale=1.0 1.0 1.0
- link LH_shank_fixed: geometry collision box size=0.114998 0.0675 0.04; collision cylinder length=0.04 radius=0.06
- link LH_thigh_fixed: geometry collision box size=0.075 0.06 0.282627; collision cylinder length=0.08 radius=0.065
- link RF_FOOT: geometry collision cylinder length=0.282504 radius=0.0175; collision sphere radius=0.03
- link RF_HAA: geometry visual mesh filename=package://legged_bringup/resource/anymal_c/meshes/drive.dae scale=1.0 1.0 1.0
- link RF_HFE: geometry collision cylinder length=0.14 radius=0.05; visual mesh filename=package://legged_bringup/resource/anymal_c/meshes/drive.dae scale=1.0 1.0 1.0
- link RF_KFE: geometry collision cylinder length=0.14 radius=0.05; visual mesh filename=package://legged_bringup/resource/anymal_c/meshes/drive.dae scale=1.0 1.0 1.0
- link RF_hip_fixed: geometry visual mesh filename=package://legged_bringup/resource/anymal_c/meshes/hip_r.dae scale=1.0 1.0 1.0
- link RF_shank_fixed: geometry collision box size=0.114998 0.0675 0.04; collision cylinder length=0.04 radius=0.06
- link RF_thigh_fixed: geometry collision box size=0.075 0.06 0.282627; collision cylinder length=0.08 radius=0.065
- link RH_FOOT: geometry collision cylinder length=0.282504 radius=0.0175; collision sphere radius=0.03
- link RH_HAA: geometry visual mesh filename=package://legged_bringup/resource/anymal_c/meshes/drive.dae scale=1.0 1.0 1.0
- link RH_HFE: geometry collision cylinder length=0.14 radius=0.05; visual mesh filename=package://legged_bringup/resource/anymal_c/meshes/drive.dae scale=1.0 1.0 1.0
- link RH_KFE: geometry collision cylinder length=0.14 radius=0.05; visual mesh filename=package://legged_bringup/resource/anymal_c/meshes/drive.dae scale=1.0 1.0 1.0
- link RH_hip_fixed: geometry visual mesh filename=package://legged_bringup/resource/anymal_c/meshes/hip_l.dae scale=1.0 1.0 1.0
- link RH_shank_fixed: geometry collision box size=0.114998 0.0675 0.04; collision cylinder length=0.04 radius=0.06
- link RH_thigh_fixed: geometry collision box size=0.075 0.06 0.282627; collision cylinder length=0.08 radius=0.065
- link base: geometry collision box size=0.58 0.14 0.18; collision cylinder length=0.145 radius=0.09
- link battery: geometry visual mesh filename=package://legged_bringup/resource/anymal_c/meshes/battery.d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 scale=1.0 1.0 1.0
- link bottom_shell: geometry visual mesh filename=package://legged_bringup/resource/anymal_c/meshes/bottom_sh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 scale=1.0 1.0 1.0
- link depth_camera_front_camera: geometry visual mesh filename=package://legged_bringup/resource/anymal_c/meshes/depth_cam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 scale=1.0 1.0 1.0
- link depth_camera_left_camera: geometry visual mesh filename=package://legged_bringup/resource/anymal_c/meshes/depth_cam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 scale=1.0 1.0 1.0
- link depth_camera_rear_camera: geometry visual mesh filename=package://legged_bringup/resource/anymal_c/meshes/depth_cam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 scale=1.0 1.0 1.0
- link depth_camera_right_camera: geometry visual mesh filename=package://legged_bringup/resource/anymal_c/meshes/depth_cam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 scale=1.0 1.0 1.0
- link face_front: geometry collision box size=0.11 0.14 0.18; collision cylinder length=0.11 radius=0.09
- link face_rear: geometry collision box size=0.11 0.14 0.18; collision cylinder length=0.11 radius=0.09
- link handle: geometry visual mesh filename=package://legged_bringup/resource/anymal_c/meshes/handle.dae scale=1.0 1.0 1.0
- link hatch: geometry visual mesh filename=package://legged_bringup/resource/anymal_c/meshes/hatch.dae scale=1.0 1.0 1.0
- link lidar: geometry visual mesh filename=package://legged_bringup/resource/anymal_c/meshes/lidar.dae
- link lidar_cage: geometry collision cylinder length=0.12 radius=0.07; visual mesh filename=package://legged_bringup/resource/anymal_c/meshes/lidar_cag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 scale=1.0 1.0 1.0
- link remote: geometry visual mesh filename=package://legged_bringup/resource/anymal_c/meshes/remote.dae scale=1.0 1.0 1.0
- link top_shell: geometry visual mesh filename=package://legged_bringup/resource/anymal_c/meshes/top_shell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 scale=1.0 1.0 1.0
- link wide_angle_camera_front_camera: geometry visual mesh filename=package://legged_bringup/resource/anymal_c/meshes/wide_angl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 scale=1.0 1.0 1.0
- link wide_angle_camera_rear_camera: geometry visual mesh filename=package://legged_bringup/resource/anymal_c/meshes/wide_angl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 scale=1.0 1.0 1.0

File: src/legged_bringup/resource/anymal_c/urdf/gazebo.xacro (robot description, xacro)
@@ -3,10 +3,71 @@
 <robot xmlns:xacro="http://www.ros.org/wiki/xacro" name="anymal">
     <xacro:include filename="anymal.urdf" />
-    <xacro:include filename="joint_gz.xacro" />
-    <xacro:leggedbot_base name="anymal" />
-    <gazebo>
-        <plugin filename="libgz_ros2_control-system.so" name="gz_ros2_control::GazeboSimROS2ControlPlugin">
-            <parameters>$(find legged_bringup)/launch/anymal.yaml</parameters>
-        </plugin>
-    </gazebo>
+    <!-- 包括机器人URDF描述 -->
+    <ros2_control name="simIMU" type="sensor">
+        <hardware>
+            <plugin>legged/simImu</plugin>
+            <param name="imu_topic">/anymal/imu</param>
+            <param name="imu_name">imu</param>
+        </hardware>
+        <sensor name="imu">
+            <state_interface name="orientation.x" />
+            <state_interface name="orientation.y" />
+            <state_interface name="orientation.z" />
+            <state_interface name="orientation.w" />
+            <state_interface name="angular_velocity.x" />
+            <state_interface name="angular_velocity.y" />
+            <state_interface name="angular_velocity.z" />
+            <state_interface name="linear_acceleration.x" />
+            <state_interface name="linear_acceleration.y" />
+            <state_interface name="linear_acceleration.z" />
+        </sensor>
+    </ros2_control>
+    <!-- 加载imu硬件 -->
+    <ros2_control name="simContact" type="sensor">
+        <hardware>
+            <plugin>legged/simContact</plugin>
+            <param name="contacts_topic_LF">/world/empty/model/anymal/link/LF_SHANK/sensor/lf_foot_contact/contact</param>
+            <param name="contacts_topic_LH">/world/empty/model/anymal/link/LH_SHANK/sensor/lh_foot_contact/contact</param>
+            <param name="contacts_topic_RF">/world/empty/model/anymal/link/RF_SHANK/sensor/rf_foot_contact/contact</param>
+            <param name="contacts_topic_RH">/world/empty/model/anymal/link/RH_SHANK/sensor/rh_foot_contact/contact</param>
+        </hardware>
+        <sensor name="contact">
+            <state_interface name="LF" data_type="bool"/>
+            <state_interface name="LH" data_type="bool"/>
+            <state_interface name="RF" data_type="bool"/>
+            <state_interface name="RH" data_type="bool"/>
+        </sensor>
+    </ros2_control>
+    <!-- 加载接触传感器硬件 -->
+    <xacro:macro name="motor" params="name">
+        <joint name="${name}">
+            <command_interface name="position" />
+            <command_interface name="velocity" />
+            <command_interface name="effort" />
+            <state_interface name="position" />
+            <state_interface name="velocity" />
+            <state_interface name="effort" />
+        </joint>
+    </xacro:macro>
+    <!-- 关节电机简化宏 -->
+    <ros2_control name="simMotor" type="system">
+        <hardware>
+            <plugin>legged/simMotor</plugin>
+            <param name="joint_state_topic">/anymal/joint/states</param>
+            <param name="joint_command_topic">/anymal/joint/cmd</param>
+        </hardware>
+        <xacro:motor name="LF_HAA" />
+        <xacro:motor name="LF_HFE" />
+        <xacro:motor name="LF_KFE" />
+        <xacro:motor name="LH_HAA" />
+        <xacro:motor name="LH_HFE" />
+        <xacro:motor name="LH_KFE" />
+        <xacro:motor name="RF_HAA" />
+        <xacro:motor name="RF_HFE" />
+        <xacro:motor name="RF_KFE" />
+        <xacro:motor name="RH_HAA" />
+        <xacro:motor name="RH_HFE" />
+        <xacro:motor name="RH_KFE" />
+    </ros2_control>
+    <!-- 加载电机硬件 -->
 </robot>
