Commit message: A1 can be launched on gazebo

File: src/legged_bringup/resource/A1/urdf/A1.urdf (robot description, URDF)
Before this commit: robot robot, 18 links, 17 joints
Links:
- link LF_calf: geometry collision box size=0.2 0.016 0.016; visual mesh filename=package://legged_bringup/resource/A1/meshes/calf.dae scale=1 1 1
- link LF_hip: geometry collision cylinder length=0.04 radius=0.046; visual mesh filename=package://legged_bringup/resource/A1/meshes/hip.dae scale=1 1 1
- link LF_thigh: geometry collision box size=0.2 0.03 0.034; collision cylinder length=0.04 radius=0.041
- link LH_calf: geometry collision box size=0.2 0.016 0.016; visual mesh filename=package://legged_bringup/resource/A1/meshes/calf.dae scale=1 1 1
- link LH_hip: geometry collision cylinder length=0.04 radius=0.046; visual mesh filename=package://legged_bringup/resource/A1/meshes/hip.dae scale=1 1 1
- link LH_thigh: geometry collision box size=0.2 0.03 0.034; collision cylinder length=0.04 radius=0.041
- link RF_calf: geometry collision box size=0.2 0.016 0.016; visual mesh filename=package://legged_bringup/resource/A1/meshes/calf.dae scale=1 1 1
- link RF_hip: geometry collision cylinder length=0.04 radius=0.046; visual mesh filename=package://legged_bringup/resource/A1/meshes/hip.dae scale=1 1 1
- link RF_thigh: geometry collision box size=0.2 0.03 0.034; collision cylinder length=0.04 radius=0.041
- link RH_calf: geometry collision box size=0.2 0.016 0.016; visual mesh filename=package://legged_bringup/resource/A1/meshes/calf.dae scale=1 1 1
- link RH_hip: geometry collision cylinder length=0.04 radius=0.046; visual mesh filename=package://legged_bringup/resource/A1/meshes/hip.dae scale=1 1 1
- link RH_thigh: geometry collision box size=0.2 0.03 0.034; collision cylinder length=0.04 radius=0.041
- link base: geometry collision box size=0.267 0.194 0.114; visual mesh filename=package://legged_bringup/resource/A1/meshes/trunk.dae scale=1 1 1

File: src/legged_bringup/resource/A1/urdf/gazebo.xacro (robot description, xacro)
@@ -28,8 +28,12 @@
         <hardware>
             <plugin>legged/simContact</plugin>
-            <param name="contacts_topic_LF">/world/2026RoboCon/model/A1/link/LF_calf/sensor/LF/contact</param>
-            <param name="contacts_topic_LH">/world/2026RoboCon/model/A1/link/LH_calf/sensor/LH/contact</param>
-            <param name="contacts_topic_RF">/world/2026RoboCon/model/A1/link/RF_calf/sensor/RF/contact</param>
-            <param name="contacts_topic_RH">/world/2026RoboCon/model/A1/link/RH_calf/sensor/RH/contact</param>
+            <param name="contacts_topic_LF">LF/touched</param>
+            <param name="contacts_topic_LH">LH/touched</param>
+            <param name="contacts_topic_RF">RF/touched</param>
+            <param name="contacts_topic_RH">RH/touched</param>
+            <param name="reset_topic_LF">/LF/enable</param>
+            <param name="reset_topic_LH">/LH/enable</param>
+            <param name="reset_topic_RF">/RF/enable</param>
+            <param name="reset_topic_RH">/RH/enable</param>
         </hardware>
         <sensor name="contact">
@@ -43,10 +47,10 @@
     <xacro:macro name="motor" params="joint_name">
         <joint name="${joint_name}">
-            <command_interface name="position" />
-            <command_interface name="velocity" />
+            <!-- <command_interface name="position" />
+            <command_interface name="velocity" /> -->
             <command_interface name="effort" />
             <state_interface name="position" />
             <state_interface name="velocity" />
-            <state_interface name="effort" />
+            <!-- <state_interface name="effort" /> -->
         </joint>
     </xacro:macro>
